Commit message: updates for figuring out starting location

File: genesis_sim2real/envs/gen3_lite_2f_robotiq_85.urdf (robot description, URDF)
Before this commit: robot gen3_lite_gen3_lite_2f, 14 links, 13 joints
Joints:
- joint left_finger_tip_joint: mimic joint=right_finger_bottom_joint multiplier=-0.676 offset=0.149 -> joint=right_finger_bottom_joint multiplier=-0.676 offset=-0.05
- joint right_finger_tip_joint: mimic joint=right_finger_bottom_joint multiplier=-0.676 offset=0.149 -> joint=right_finger_bottom_joint multiplier=-0.676 offset=-0.05
